Commit message: Simulation: 16-beam lidar, encoder odometry, lidar odometry in the EKF, simple_env1 world

File: ros2_packages/scout_nav2/agilex_scout/urdf/mobile_robot/scout_v2.urdf.xacro (robot description, xacro)
@@ -48,19 +48,16 @@
 			</collision>
 		</link>
-		<link name="inertial_link">
+		<!-- <link name="inertial_link">
 			<inertial>
 				<mass value="50" />
-				<!-- <mass value="50" /> -->
-				<!-- <origin xyz="-0.00065 -0.085 0.062" />
-			<inertia ixx="0.6022" ixy="-0.02364" ixz="-0.1197" iyy="1.7386" iyz="-0.001544" izz="2.0296" /> -->
 				<origin xyz="0.0 0.0 0.0" />
 				<inertia ixx="2.288641" ixy="0" ixz="0" iyy="5.103976" iyz="0" izz="3.431465" />
 			</inertial>
-		</link>
-		<joint name="inertial_joint" type="fixed">
+		</link> -->
+		<!-- <joint name="inertial_joint" type="fixed">
 			<origin xyz="0 0 0" rpy="0 0 0" />
 			<parent link="mobile_robot_base_link" />
 			<child link="inertial_link" />
-		</joint>
+		</joint> -->
 		<!-- Scout wheel macros -->
 		<xacro:include filename="$(find agilex_scout)/urdf/mobile_robot/scout_wheel_type1.xacro" />
